File: 01.ActJIS104/02.Assemble/ActJIS104.kicad_pcb (KiCad board)
At the start: 2 copper layers, 304.4 x 98.8 mm, 136 parts, among them J1 Conn_01x02, J11 Conn_01x01, J12 Conn_01x01, SW1 SW_PUSH, SW10 SW_PUSH, SW11 SW_PUSH, SW12 SW_PUSH, SW13 SW_PUSH, SW14 SW_PUSH, SW15 SW_PUSH, SW16 SW_PUSH, SW17 SW_PUSH, SW18 SW_PUSH, SW19 SW_PUSH, SW2 SW_PUSH, SW20 SW_PUSH, SW21 SW_PUSH, SW22 SW_PUSH, SW23 SW_PUSH, SW24 SW_PUSH, SW25 SW_PUSH, SW26 SW_PUSH, SW27 SW_PUSH, SW28 SW_PUSH, SW29 SW_PUSH, SW3 SW_PUSH, SW30 SW_PUSH, SW31 SW_PUSH, SW32 SW_PUSH, SW33 SW_PUSH, SW34 SW_PUSH, SW35 SW_PUSH, SW36 SW_PUSH, SW37 SW_PUSH, SW38 SW_PUSH, SW39 SW_PUSH, SW4 SW_PUSH, SW40 SW_PUSH, SW41 SW_PUSH, SW42 SW_PUSH, SW43 SW_PUSH, SW44 SW_PUSH, SW45 SW_PUSH, SW46 SW_PUSH, SW47 SW_PUSH, SW48 SW_PUSH, SW49 SW_PUSH, SW5 SW_PUSH, SW50 SW_PUSH, SW51 SW_PUSH, SW52 SW_PUSH, SW53 SW_PUSH, SW54 SW_PUSH, SW55 SW_PUSH, SW56 SW_PUSH, SW57 SW_PUSH, SW58 SW_PUSH, SW59 SW_PUSH, SW6 SW_PUSH, SW60 SW_PUSH, SW61 SW_PUSH, SW62 SW_PUSH, SW63 SW_PUSH, SW64 SW_PUSH, SW65 SW_PUSH, SW66 SW_PUSH, SW7 SW_PUSH, SW8 SW_PUSH, SW9 SW_PUSH, U1 BLEMicroPro

Commit message: Add files via upload
Parts:
- SW1, SW7: footprint kbd_SW:CherryMX_Hotswap_1u -> kbd_SW:CherryMX_Hotswap_1u_Small1
- SW28: footprint kbd_SW:CherryMX_Hotswap_6.25u -> kbd_SW:CherryMX_Hotswap_6.25u_Rev
- SW4, SW61: footprint kbd_SW:CherryMX_Hotswap_2.25u -> kbd_SW:CherryMX_Hotswap_2.25u_Rev
- SW62: footprint kbd_SW:CherryMX_Hotswap_2.75u -> kbd_SW:CherryMX_Hotswap_2.75u_Rev
- moved D64 19.1 mm to (285.8, 35.7)
- moved D7 14.5 mm to (66.7, 35.7)
- moved D28 14.3 mm to (150.0, 111.9)
- moved D4 14.3 mm to (40.5, 92.9)
- moved D62 14.3 mm to (297.7, 92.9)
- moved D61 14.3 mm to (302.4, 73.8)
- moved D12 9.53 mm to (76.2, 35.7)
- moved D1 4.80 mm to (32.7, 38.1)
Routing:
- net Col6: track 502.6 -> 462.1 mm
- net Row4: track 455.9 -> 428.2 mm
- net Net-(D64-Pad1): track 23.6 -> 46.1 mm
- net Row0: track 345.9 -> 326.1 mm, vias 2 -> 4
- net Col0: track 378.4 -> 360.3 mm, vias 13 -> 9
- net Net-(D7-Pad2): track 13.5 -> 28.3 mm
- net Row3: track 403.9 -> 411.3 mm, vias 1 -> 2
- net Net-(D62-Pad1): track 16.5 -> 23.6 mm
- net Net-(D61-Pad1): track 17.1 -> 23.6 mm
- net Net-(D28-Pad2): track 23.1 -> 16.8 mm
- net Net-(D4-Pad2): track 23.1 -> 16.8 mm
- net Row2: track 404.0 -> 398.1 mm
- net Net-(D1-Pad2): track 13.7 -> 18.7 mm
- net Reset: track 34.8 -> 30.4 mm, vias 4 -> 3
- net Col4: track 354.8 -> 357.2 mm, vias 13 -> 14
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