File: 01.ActJIS104/03.Decoration/ActJIS104.kicad_pcb (KiCad board)
At the start: 2 copper layers, 325.8 x 112.2 mm, 10 parts, among them J10 Conn_01x01, J11 Conn_01x01, J12 Conn_01x01, J13 Conn_01x01, J14 Conn_01x01, J15 Conn_01x01, J16 Conn_01x01, J17 Conn_01x01, J8 Conn_01x01, J9 Conn_01x01

Commit message: Add files via upload
Parts:
- J11, J12, J13: footprint kbd_Hole:m2_Screw_Hole_Fab -> kbd_Hole:m2_Screw_Hole_EdgeCuts
Other:
- outline, holes or cut-outs redrawn
Changed lines of the file:
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@@
       (drillshape 0)
       (scaleselection 1)
-      (outputdirectory "C:/Users/サリチル酸/Desktop/")
+      (outputdirectory "../04.発注/02.Decoration/")
     )
   )
@@
     (fp_circle (center 0 0) (end 1.1 0) (layer "Edge.Cuts") (width 0.01) (fill none))
   )
-  (footprint "kbd_Hole:m2_Screw_Hole_Fab" (layer "F.Cu")
+  (footprint "kbd_Hole:m2_Screw_Hole_EdgeCuts" (layer "F.Cu")
     (at 108.575 13.05)
     (descr "Mounting Hole 2.2mm, no annular, M2")
@@
       (effects (font (size 1 1) (thickness 0.15)))
     )
-    (fp_circle (center 0 0) (end 1.1 0) (layer "F.Fab") (width 0.01) (fill none))
+    (fp_circle (center 0 0) (end 1.1 0) (layer "Edge.Cuts") (width 0.01) (fill none))
   )
-  (footprint "kbd_Hole:m2_Screw_Hole_Fab" (layer "F.Cu")
+  (footprint "kbd_Hole:m2_Screw_Hole_EdgeCuts" (layer "F.Cu")
     (at 234.325 13.05)
     (descr "Mounting Hole 2.2mm, no annular, M2")
@@
       (effects (font (size 1 1) (thickness 0.15)))
     )
-    (fp_circle (center 0 0) (end 1.1 0) (layer "F.Fab") (width 0.01) (fill none))
+    (fp_circle (center 0 0) (end 1.1 0) (layer "Edge.Cuts") (width 0.01) (fill none))
   )
-  (footprint "kbd_Hole:m2_Screw_Hole_Fab" (layer "F.Cu")
+  (footprint "kbd_Hole:m2_Screw_Hole_EdgeCuts" (layer "F.Cu")
     (at 108.575 120.25)
     (descr "Mounting Hole 2.2mm, no annular, M2")
@@
       (effects (font (size 1 1) (thickness 0.15)))
     )
-    (fp_circle (center 0 0) (end 1.1 0) (layer "F.Fab") (width 0.01) (fill none))
+    (fp_circle (center 0 0) (end 1.1 0) (layer "Edge.Cuts") (width 0.01) (fill none))
   )
   (footprint "kbd_Hole:m2_Screw_Hole_EdgeCuts" (layer "F.Cu")
@@
   (gr_line (start 334.325 121.25) (end 334.325 12.05) (layer "Edge.Cuts") (width 0.15))
   (gr_line (start 323.35 114.3) (end 267.2 114.3) (layer "Edge.Cuts") (width 0.1))
-  (gr_circle (center 314.325 47.625) (end 314.4 41.625) (layer "Edge.Cuts") (width 0.1) (fill none))
   (gr_line (start 323.35 38.1) (end 305.3 38.1) (layer "Edge.Cuts") (width 0.1))
   (gr_arc (start 323.35 57.15) (mid 323.703553 57.296447) (end 323.85 57.65) (layer "Edge.Cuts") (width 0.1))
